Commit message: Add base_footprint link

File: ackermann_vehicle/ackermann_vehicle_description/urdf/em_3905.urdf.xacro (robot description, xacro)
@@ -301,4 +301,5 @@
        rviz. -->
   <link name="base_link" />
+  <link name="base_footprint" />
   <!-- Chassis -->
   <link name="chassis">
@@ -328,4 +329,9 @@
     <parent link="base_link"/>
     <child link="chassis"/>
+  </joint>
+  <joint name="base_footprint_to_link" type="fixed">
+    <parent link="base_footprint"/>
+    <child link="base_link"/>
+    <origin xyz="0 0 0.1" />
   </joint>
   <!-- Batteries -->
@@ -366,5 +372,5 @@
     <plugin name="gazebo_ros_p3d"     filename="libgazebo_ros_p3d.so">
       <frameName>map</frameName>
-      <bodyName>base_link</bodyName>
+      <bodyName>base_footprint</bodyName>
       <topicName>odom_truth</topicName>
       <updateRate>30.0</updateRate>
